File: HW/Lab10_Starter.sch (EAGLE design)
At the start: 13 parts, among them IC1 OPA4350P, Q1 IRLD024

Commit message: py script comm
Parts:
- removed IC1: OPA4350P, EE445L:OPA4350P
- removed R3, R4: 10k, EE445L:RESISTOR0204/5
- removed R5: 200k, EE445L:RESISTOR0204/5
- C1: value .1uf -> 1uf; device EE445L:CAPACITOR025-024X044 -> EE445L:CAPACITOR050-024X044
Connections:
- removed net A: JP1.4
- removed net M2: JP1.2
- removed net N$3: D1.A, Q1.D
- removed net N$4: R2.2, R3.1, R4.2
- removed net N$5: IC1A.+IN, R4.1, R5.2
- net +3V3: now also R2.2; no longer C1.1, IC1A.V+, R3.2
- net +5V: now also JP1.2
- net GND: no longer IC1A.V-, R2.1
- net M1: now also D1.A, Q1.D
- net N$2: now also C1.1
- net TACH: now also JP1.4, R2.1; no longer IC1A.OUT, R5.1
Other:
- moved on the sheet: C1, R1, R2
